File: Hardware/InkTime-SmartWatch.brd (EAGLE design)
At the start: 46 x 35 mm, 105 parts, among them IC1 BQ25180YBGR, IC2 DRV2605YZFR, IC3 BMA421, IC9 RT6160AWSC, J1 503480-2400, J2 TC2030-IDC, J4 KH-TYPE-C-16P, Q1 20V/4.2A/52mΩ/1.4W, Q3 SI1308EDL-T1-GE3, U1 NRF52840_QF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

Commit message: Add files via upload
Parts:
- moved TP_SDA 17.0 mm to (17.1, 7.66)
- moved TP_SCL 11.5 mm to (27.6, 7.94)
- moved TP_ON 8.09 mm to (30.7, 6.89)
- moved R3 2.11 mm to (16.1, 10.2)
- moved C21 2.10 mm to (34.8, 17.3), turned to 270 degrees
- moved EPD_C5 1.90 mm to (26.7, 23.0)
- moved C6 1.85 mm to (29.5, 23.1)
- moved D5 1.66 mm to (20.3, 38.6)
- moved TP_VBAT 1.62 mm to (42.0, 9.35)
- moved EPD_C6 1.56 mm to (26.4, 22.1)
- moved EPD_C11 1.53 mm to (26.9, 16.3), turned to 90 degrees
- moved C1 1.30 mm to (46.0, 25.4)
- moved EPD_C7 1.23 mm to (26.4, 21.1)
- moved C7 1.21 mm to (38.4, 18.2)
- moved C10 1.14 mm to (42.6, 24.8), turned to 270 degrees
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Routing:
- net 3V3: track 24.4 -> 166.6 mm, vias 0 -> 22
- net SCL: track 1.15 -> 112.7 mm, vias 0 -> 17
- net SDA: track 1.13 -> 88.5 mm, vias 0 -> 12
- net VREG: track 9.12 -> 55.3 mm, vias 0 -> 4
- net EPD_RST: track 0.00 -> 43.9 mm, vias 0 -> 12
- net ALERT: track 0.00 -> 40.9 mm, vias 0 -> 10
- net VBUS: track 17.8 -> 58.7 mm, vias 0 -> 6
- net D-: track 0.00 -> 28.9 mm, vias 0 -> 4
- net RESET: track 5.63 -> 31.9 mm, vias 0 -> 8
- net EPD_3V3: track 9.17 -> 33.9 mm, vias 0 -> 3
- net D+: track 0.00 -> 24.6 mm, vias 0 -> 2
- net PREVGH: track 2.29 -> 26.6 mm, vias 0 -> 2
- net MOSI: track 0.00 -> 24.0 mm, vias 0 -> 4
- net SCK: track 0.00 -> 23.2 mm, vias 0 -> 2
- net IMU_INT2: track 0.00 -> 23.1 mm, vias 0 -> 2
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- added copper zone on layer 1, net GND
Other:
- outline, holes or cut-outs redrawn

Commit message: Varianta finala de PCB 2D
Parts:
- moved TP_SDA 2.03 mm to (19.0, 8.22)
- moved EPD_C11 1.00 mm to (25.9, 16.5)
- moved EPD_C10 0.74 mm to (25.1, 18.0)
- moved TP_OP 0.72 mm to (25.6, 13.5)
- moved EPD_C12 0.51 mm to (24.9, 15.5), turned to 90 degrees
- moved C42 0.49 mm to (34.7, 32.2)
- moved C5 0.43 mm to (31.8, 26.6)
- moved C32 0.42 mm to (27.6, 13.5)
- moved C9 0.38 mm to (41.7, 22.6)
- moved C18 0.36 mm to (28.0, 25.1), turned to 90 degrees
- moved C6 0.30 mm to (29.5, 22.8)
- moved C15 0.29 mm to (35.3, 27.9)
- moved C27 0.26 mm to (28.0, 17.4)
- moved R1_USB 0.26 mm to (40.1, 32.5), turned to 0 degrees
- moved C7 0.25 mm to (38.3, 17.9)
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Routing:
- net GND: track 7.01 -> 168.3 mm, vias 0 -> 33
- net 3V3: track 166.6 -> 168.9 mm
- net SDA: track 88.5 -> 90.6 mm
- net SWDIO: track 11.8 -> 13.7 mm
- net N$19: track 16.4 -> 18.1 mm, vias 2 -> 4
- net VBUS: track 58.7 -> 60.2 mm
- net N$3: track 7.11 -> 8.56 mm, vias 0 -> 2
- net OUT+: track 4.22 -> 5.57 mm
- net VREG: track 55.3 -> 56.5 mm
- net LX1: track 2.74 -> 3.92 mm
- net OUT-: track 11.4 -> 12.5 mm
- net P1.01: track 19.7 -> 20.6 mm
- net PMIC_INT: track 16.7 -> 17.5 mm
- net SWDCLK: track 16.2 -> 17.0 mm
- net N$26: track 2.43 -> 1.73 mm
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- added copper zone on layer 16, net GND
